Commit message: Updated ordering

File: eeduro_delta_description/urdf/eeduro_delta.urdf.xacro (robot description, xacro)
@@ -31,4 +31,96 @@
 		<xacro:base_inertial/>
 	</link>
+    	<!-- x y z are the center of the robot, in the high:of the mounting-points for the arms -->
+	<xacro:macro name="delta_arm" params="parent arm_end_child arm_nr joint4_type angle1 angle2 angle3 dist_xy x y z roll pitch yaw">
+		<joint name="arm${arm_nr}_motor_joint" type="continuous">
+		  <parent link="${parent}"/>
+		  <child link="arm${arm_nr}_motor"/>
+		  <origin xyz="${x +cos(yaw)*dist_xy -sin(yaw)*(0.04)} ${y +sin(yaw)*dist_xy +cos(yaw)*(0.04)} ${z -0.015}" rpy="${roll -pi/2} ${pitch} ${yaw -pi/2}"/>
+		  <axis xyz="1 0 0"/>
+		  <dynamics damping="0.0000001"/>
+		</joint>
+		<link name="arm${arm_nr}_motor">
+	  <visual>
+	    <origin xyz="0 0 0" rpy="0 ${pi/2} 0"/>
+	    <geometry>
+	      <cylinder radius="0.006" length="0.018"/>
+	    </geometry>
+	  </visual>
+		<xacro:motor_inertial/>
+		</link>
+		<joint name="arm${arm_nr}_joint0" type="continuous">
+		  <parent link="${parent}"/>
+		  <child link="arm${arm_nr}_link1"/>
+		  <!-- callculation X: 0  Y: -70.23..+17.5  Z: 210-15 -->
+		  <origin xyz="${x +cos(yaw)*dist_xy} ${y +sin(yaw)*dist_xy}  ${z -0.015}" rpy="${roll -pi/2  +angle1} ${pitch} ${yaw -pi/2}"/>
+		  <axis xyz="1 0 0"/>
+		  <dynamics damping="0.0001"/>
+		</joint>
+		<link name="arm${arm_nr}_link1">
+		  <visual>
+		    <origin xyz="0 0 0" rpy="0 0 0"/>
+		    <geometry>
+		      <mesh filename="package://eeduro_delta_description/meshes/link1_scaled.dae"/>
+		    </geometry>
+		  </visual>
+			<collision>
+				<origin xyz="0 0 0.024" rpy="0 0 0"/>
+				<geometry>
+					<box size="0.006 0.012 0.06 "/>
+				</geometry>
+			</collision>
+			<xacro:link1_inertial/>
+		</link>
+		<gazebo>
+		  <joint name="arm${arm_nr}_gearbox" type="gearbox">
+		    <parent>arm${arm_nr}_motor</parent>
+		    <child>arm${arm_nr}_link1</child>
+		    <gearbox_reference_body>${parent}</gearbox_reference_body>
+		    <gearbox_ratio>-0.013176411</gearbox_ratio>
+		    <axis>
+					<use_parent_model_frame>false</use_parent_model_frame>
+		      <xyz>1 0 0</xyz>
+		    </axis>
+		    <axis2>
+					<use_parent_model_frame>false</use_parent_model_frame>
+		      <xyz>1 0 0</xyz>
+		    </axis2>
+		  </joint>
+		</gazebo>
+		<joint name="arm${arm_nr}_joint1" type="continuous">
+		  <parent link="arm${arm_nr}_link1"/>
+		  <child link="arm${arm_nr}_link2"/>
+		  <origin xyz="0 0 0.05" rpy="${angle2} 0 0"/>
+		  <axis xyz="1 0 0"/>
+		  <dynamics damping="0.00001"/>
+		</joint>
+		<link name="arm${arm_nr}_link2">
+		  <visual>
+		    <origin xyz="0 0 0" rpy="0 0 0"/>
+		    <geometry>
+		      <mesh filename="package://eeduro_delta_description/meshes/link2_scaled.dae"/>
+		    </geometry>
+		  </visual>
+			<collision>
+		    <origin xyz="0 0 0" rpy="0 0 0"/>
+		    <geometry>
+					<box size="0.044 0.008 0.006"/>
+				</geometry>
+			</collision>
+			<xacro:link2_inertial/>
+		</link>
+		<xacro:link3_with_joint arm_nr="${arm_nr}" suffix="_1" sign="+" joint3_type="urdf"/>
+		<xacro:link3_with_joint arm_nr="${arm_nr}" suffix="_2" sign="-" joint3_type="sdf"/>
+		<link name="arm${arm_nr}_link4">
+		  <visual>
+		    <origin xyz="0 -0.018 0" rpy="0 0 ${pi/2}"/>
+		    <geometry>
+		      <mesh filename="package://eeduro_delta_description/meshes/link2_scaled.dae"/>
+		    </geometry>
+		  </visual>
+			<xacro:link4_inertial/>
+		</link>
+		<xacro:element xacro:name="joint4_${joint4_type}" arm_nr="${arm_nr}" child="${arm_end_child}" angle="${angle3}"/>
+	</xacro:macro>
 	<xacro:delta_arm
 		parent="base_link"
@@ -106,96 +198,4 @@
 	  <selfCollide>true</selfCollide>
 	</gazebo>
-	<!-- x y z are the center of the robot, in the high:of the mounting-points for the arms -->
-	<xacro:macro name="delta_arm" params="parent arm_end_child arm_nr joint4_type angle1 angle2 angle3 dist_xy x y z roll pitch yaw">
-		<joint name="arm${arm_nr}_motor_joint" type="continuous">
-		  <parent link="${parent}"/>
-		  <child link="arm${arm_nr}_motor"/>
-		  <origin xyz="${x +cos(yaw)*dist_xy -sin(yaw)*(0.04)} ${y +sin(yaw)*dist_xy +cos(yaw)*(0.04)} ${z -0.015}" rpy="${roll -pi/2} ${pitch} ${yaw -pi/2}"/>
-		  <axis xyz="1 0 0"/>
-		  <dynamics damping="0.0000001"/>
-		</joint>
-		<link name="arm${arm_nr}_motor">
-	  <visual>
-	    <origin xyz="0 0 0" rpy="0 ${pi/2} 0"/>
-	    <geometry>
-	      <cylinder radius="0.006" length="0.018"/>
-	    </geometry>
-	  </visual>
-		<xacro:motor_inertial/>
-		</link>
-		<joint name="arm${arm_nr}_joint0" type="continuous">
-		  <parent link="${parent}"/>
-		  <child link="arm${arm_nr}_link1"/>
-		  <!-- callculation X: 0  Y: -70.23..+17.5  Z: 210-15 -->
-		  <origin xyz="${x +cos(yaw)*dist_xy} ${y +sin(yaw)*dist_xy}  ${z -0.015}" rpy="${roll -pi/2  +angle1} ${pitch} ${yaw -pi/2}"/>
-		  <axis xyz="1 0 0"/>
-		  <dynamics damping="0.0001"/>
-		</joint>
-		<link name="arm${arm_nr}_link1">
-		  <visual>
-		    <origin xyz="0 0 0" rpy="0 0 0"/>
-		    <geometry>
-		      <mesh filename="package://eeduro_delta_description/meshes/link1_scaled.dae"/>
-		    </geometry>
-		  </visual>
-			<collision>
-				<origin xyz="0 0 0.024" rpy="0 0 0"/>
-				<geometry>
-					<box size="0.006 0.012 0.06 "/>
-				</geometry>
-			</collision>
-			<xacro:link1_inertial/>
-		</link>
-		<gazebo>
-		  <joint name="arm${arm_nr}_gearbox" type="gearbox">
-		    <parent>arm${arm_nr}_motor</parent>
-		    <child>arm${arm_nr}_link1</child>
-		    <gearbox_reference_body>${parent}</gearbox_reference_body>
-		    <gearbox_ratio>-0.013176411</gearbox_ratio>
-		    <axis>
-					<use_parent_model_frame>false</use_parent_model_frame>
-		      <xyz>1 0 0</xyz>
-		    </axis>
-		    <axis2>
-					<use_parent_model_frame>false</use_parent_model_frame>
-		      <xyz>1 0 0</xyz>
-		    </axis2>
-		  </joint>
-		</gazebo>
-		<joint name="arm${arm_nr}_joint1" type="continuous">
-		  <parent link="arm${arm_nr}_link1"/>
-		  <child link="arm${arm_nr}_link2"/>
-		  <origin xyz="0 0 0.05" rpy="${angle2} 0 0"/>
-		  <axis xyz="1 0 0"/>
-		  <dynamics damping="0.00001"/>
-		</joint>
-		<link name="arm${arm_nr}_link2">
-		  <visual>
-		    <origin xyz="0 0 0" rpy="0 0 0"/>
-		    <geometry>
-		      <mesh filename="package://eeduro_delta_description/meshes/link2_scaled.dae"/>
-		    </geometry>
-		  </visual>
-			<collision>
-		    <origin xyz="0 0 0" rpy="0 0 0"/>
-		    <geometry>
-					<box size="0.044 0.008 0.006"/>
-				</geometry>
-			</collision>
-			<xacro:link2_inertial/>
-		</link>
-		<xacro:link3_with_joint arm_nr="${arm_nr}" suffix="_1" sign="+" joint3_type="urdf"/>
-		<xacro:link3_with_joint arm_nr="${arm_nr}" suffix="_2" sign="-" joint3_type="sdf"/>
-		<link name="arm${arm_nr}_link4">
-		  <visual>
-		    <origin xyz="0 -0.018 0" rpy="0 0 ${pi/2}"/>
-		    <geometry>
-		      <mesh filename="package://eeduro_delta_description/meshes/link2_scaled.dae"/>
-		    </geometry>
-		  </visual>
-			<xacro:link4_inertial/>
-		</link>
-		<xacro:element xacro:name="joint4_${joint4_type}" arm_nr="${arm_nr}" child="${arm_end_child}" angle="${angle3}"/>
-	</xacro:macro>
 	<xacro:macro name="link3_with_joint" params="arm_nr suffix sign joint3_type">
 		<joint name="arm${arm_nr}_joint2${suffix}" type="continuous">

File: eeduro_delta_description/urdf/eeduro_delta_inertial.urdf.xacro (robot description, xacro)
@@ -1,84 +1,65 @@
 <?xml version="1.0"?>
-<robot name="eeduro_delta" xmlns:xacro="http://www.ros.org/wiki/xacro">
-	<xacro:macro name="base_inertial">
-		<inertial>
-			<origin		xyz="	-3.61483029333e-10
+<robot name="eeduro_delta"
+    xmlns:xacro="http://www.ros.org/wiki/xacro">
+    <xacro:macro name="base_inertial">
+        <inertial>
+            <origin xyz="	-3.61483029333e-10
 											 0.0127334577336
-											 0.0879729092856"
-								rpy="0 0 0"/>
-			<mass value="1.9"/>
-			<inertia  ixx="0.02085588597106"			ixy="-1.660569664432e-10"		ixz="-1.1398676896544e-10"
-																						iyy="0.02129590096144"			iyz="0.0016993275934572"
-																																				izz="0.019156198852616"/>
-		</inertial>
-	</xacro:macro>
-	<xacro:macro name="motor_inertial">
-		<inertial>
-      <origin		xyz="0 0 0" rpy="0 0 0"/>
-      <mass value="0.01"/>
-      <inertia	ixx="6.5e-8"								ixy="0"											ixz="0"
-																						iyy="8.5e-8"								iyz="0"
-																																				izz="8.5e-8"/>
-    </inertial>
-	</xacro:macro>
-	<xacro:macro name="link1_inertial">
-		<inertial>
-	    <origin		xyz="	-0.000667579518792749
+											 0.0879729092856" rpy="0 0 0"/>
+            <mass value="1.9"/>
+            <inertia ixx="0.02085588597106" ixy="-1.660569664432e-10" ixz="-1.1398676896544e-10" iyy="0.02129590096144" iyz="0.0016993275934572" izz="0.019156198852616"/>
+        </inertial>
+    </xacro:macro>
+    <xacro:macro name="motor_inertial">
+        <inertial>
+            <origin xyz="0 0 0" rpy="0 0 0"/>
+            <mass value="0.01"/>
+            <inertia ixx="6.5e-8" ixy="0" ixz="0" iyy="8.5e-8" iyz="0" izz="8.5e-8"/>
+        </inertial>
+    </xacro:macro>
+    <xacro:macro name="link1_inertial">
+        <inertial>
+            <origin xyz="	-0.000667579518792749
 											 4.24024711964181e-05
-											 0.0237382053187016"
-								rpy="0 0 0"/>
-	    <mass value="0.01225732594264"/>
-	    <inertia  ixx="3.9170528247202e-06"		ixy="6.88244852580979e-11"	ixz="-4.1443351708254e-08"
-																						iyy="3.81032017743918e-06"	iyz="1.23377194660718e-08"
-																																				izz="1.78939838618822e-07"/>
-	  </inertial>
-	</xacro:macro>
-	<xacro:macro name="link2_inertial">
-		<inertial>
-	    <origin		xyz="	-4.65883028011777e-16
+											 0.0237382053187016" rpy="0 0 0"/>
+            <mass value="0.01225732594264"/>
+            <inertia ixx="3.9170528247202e-06" ixy="6.88244852580979e-11" ixz="-4.1443351708254e-08" iyy="3.81032017743918e-06" iyz="1.23377194660718e-08" izz="1.78939838618822e-07"/>
+        </inertial>
+    </xacro:macro>
+    <xacro:macro name="link2_inertial">
+        <inertial>
+            <origin xyz="	-4.65883028011777e-16
 											 0.000173858781653159
-											 5.67176538207829e-17"
-								rpy="0 0 0"/>
-	    <mass value="0.002676077437253"/>
-	    <inertia  ixx="2.12767184543771e-08"	ixy="-5.53089204125579e-22"	ixz="-3.40282030897929e-10"
-																						iyy="5.08472734636316e-07"	iyz="1.63502204451954e-23"
-																																				izz="5.19396055186747e-07"/>
-	  </inertial>
-	</xacro:macro>
-	<xacro:macro name="link3_inertial">
-		<inertial>
-	    <origin		xyz="	4.79435653399733e-15
+											 5.67176538207829e-17" rpy="0 0 0"/>
+            <mass value="0.002676077437253"/>
+            <inertia ixx="2.12767184543771e-08" ixy="-5.53089204125579e-22" ixz="-3.40282030897929e-10" iyy="5.08472734636316e-07" iyz="1.63502204451954e-23" izz="5.19396055186747e-07"/>
+        </inertial>
+    </xacro:macro>
+    <xacro:macro name="link3_inertial">
+        <inertial>
+            <origin xyz="	4.79435653399733e-15
 											5.05515762210611e-15
-											0.05"
-								rpy="0 0 0"/>
-	    <mass value="0.00303456300894497"/>
-	    <inertia  ixx="3.21114513230401e-06"	ixy="-1.39831896086795e-22"	ixz="-1.65818121965606e-19"
-																						iyy="3.20896476471281e-06"	iyz="-7.25104237772119e-20"
-																																				izz="5.81686125403351e-09"/>
-	  </inertial>
-	</xacro:macro>
-	<xacro:macro name="link4_inertial">
-		<inertial>
-	    <origin		xyz="	-0.00017385878165316
+											0.05" rpy="0 0 0"/>
+            <mass value="0.00303456300894497"/>
+            <inertia ixx="3.21114513230401e-06" ixy="-1.39831896086795e-22" ixz="-1.65818121965606e-19" iyy="3.20896476471281e-06" iyz="-7.25104237772119e-20" izz="5.81686125403351e-09"/>
+        </inertial>
+    </xacro:macro>
+    <xacro:macro name="link4_inertial">
+        <inertial>
+            <origin xyz="	-0.00017385878165316
 											-0.0179999999999995
-											-5.56154717015503e-17"
-								rpy="0 0 0"/>
-	    <mass value="0.002676077437253"/>
-	    <inertia  ixx="5.08472734636316e-07"	ixy="-5.82921356214306e-22"	ixz="1.63293841801982e-23"
-																						iyy="2.12767184543771e-08"	iyz="-3.40282030897868e-10"
-																																				izz="5.19396055186747e-07"/>
-	  </inertial>
-	</xacro:macro>
-	<xacro:macro name="tool_inertial">
-		<inertial>
-	    <origin		xyz="	2.59861008225168e-05
+											-5.56154717015503e-17" rpy="0 0 0"/>
+            <mass value="0.002676077437253"/>
+            <inertia ixx="5.08472734636316e-07" ixy="-5.82921356214306e-22" ixz="1.63293841801982e-23" iyy="2.12767184543771e-08" iyz="-3.40282030897868e-10" izz="5.19396055186747e-07"/>
+        </inertial>
+    </xacro:macro>
+    <xacro:macro name="tool_inertial">
+        <inertial>
+            <origin xyz="	2.59861008225168e-05
 											0.00192804788388403
-											0.022995128907788"
-								rpy="0 0 0"/>
-	    <mass value="0.05741035631797"/>
-	    <inertia  ixx="1.98534599648007e-05"	ixy="-5.03744139689366e-09"	ixz="8.28383830393447e-10"
-																						iyy="5.51924419052098e-06"	iyz="1.3955126250812e-08"
-																																				izz="1.98271230263828e-05"/>
-	  </inertial>
-	</xacro:macro>
+											0.022995128907788" rpy="0 0 0"/>
+            <mass value="0.05741035631797"/>
+            <inertia ixx="1.98534599648007e-05" ixy="-5.03744139689366e-09" ixz="8.28383830393447e-10" iyy="5.51924419052098e-06" iyz="1.3955126250812e-08" izz="1.98271230263828e-05"/>
+        </inertial>
+    </xacro:macro>
 </robot>

Commit message: More xacro order fixes

File: eeduro_delta_description/urdf/eeduro_delta.urdf.xacro (robot description, xacro)
@@ -123,4 +123,85 @@
 		<xacro:element xacro:name="joint4_${joint4_type}" arm_nr="${arm_nr}" child="${arm_end_child}" angle="${angle3}"/>
 	</xacro:macro>
+	<xacro:macro name="link3_with_joint" params="arm_nr suffix sign joint3_type">
+		<joint name="arm${arm_nr}_joint2${suffix}" type="continuous">
+		  <parent link="arm${arm_nr}_link2"/>
+		  <child link="arm${arm_nr}_link3${suffix}"/>
+		  <origin xyz="${sign}0.018 0 0" rpy="0 0 ${-pi/2}"/>
+		  <axis xyz="1 0 0"/>
+		  <dynamics damping="0.00001"/>
+			<xacro:if value="${suffix == '_2'}">
+				<mimic joint="arm${arm_nr}_joint2_1" multiplier="1" offset="0"/>
+			</xacro:if>
+		</joint>
+		<link name="arm${arm_nr}_link3${suffix}">
+		  <visual>
+		    <origin xyz="0 0 0" rpy="0 0 0"/>
+		    <geometry>
+		      <mesh filename="package://eeduro_delta_description/meshes/link3_scaled.dae"/>
+		    </geometry>
+		  </visual>
+			<xacro:link3_inertial/>
+		</link>
+		<xacro:element xacro:name="joint3_${joint3_type}" arm_nr="${arm_nr}" suffix="${suffix}"/>
+	</xacro:macro>
+	<xacro:macro name="joint3_urdf" params="arm_nr suffix">
+			<joint name="arm${arm_nr}_joint3${suffix}" type="continuous">
+			  <parent link="arm${arm_nr}_link3${suffix}"/>
+			  <child link="arm${arm_nr}_link4"/>
+			  <origin xyz="0 0 0.1" rpy="0 0 0"/>
+			  <axis xyz="1 0 0"/>
+			  <dynamics damping="0.00001"/>
+				<mimic joint="arm${arm_nr}_joint2_1" multiplier="-1" offset="0"/>
+			</joint>
+	</xacro:macro>
+	<xacro:macro name="joint3_sdf" params="arm_nr suffix">
+		<gazebo>
+			<joint name="arm${arm_nr}_joint3${suffix}" type="revolute">
+			  <child>arm${arm_nr}_link4</child>
+			  <parent>arm${arm_nr}_link3${suffix}</parent>
+			  <pose>0 -0.036 0 0 0 0</pose>
+			  <axis>
+			    <use_parent_model_frame>false</use_parent_model_frame>
+			    <xyz>1 0 0</xyz>
+			    <limit>
+			      <lower>-1e+16</lower>
+			      <upper>1e+16</upper>
+			    </limit>
+			    <dynamics>
+			      <damping>0.00001</damping>
+			    </dynamics>
+			  </axis>
+			</joint>
+		</gazebo>
+  </xacro:macro>
+	<xacro:macro name="joint4_urdf" params="arm_nr child angle">
+		<joint name="arm${arm_nr}_joint4" type="continuous">
+		  <parent link="arm${arm_nr}_link4"/>
+		  <child link="${child}"/>
+		  <origin xyz="0 -0.018 0" rpy="${angle} 0 ${pi/2}"/>
+		  <axis xyz="1 0 0"/>
+		  <dynamics damping="0.00001"/>
+		</joint>
+	</xacro:macro>
+  <xacro:macro name="joint4_sdf" params="arm_nr child angle">
+    <gazebo>
+			<joint name="arm${arm_nr}_joint4" type="revolute">
+	      <parent>${child}</parent>
+	      <child>arm${arm_nr}_link4</child>
+	      <pose>0 -0.018 0 ${angle} 0 ${pi/2}</pose>
+				<axis>
+          <use_parent_model_frame>false</use_parent_model_frame>
+          <xyz>1 0 0</xyz>
+          <limit>
+            <lower>-1e+16</lower>
+            <upper>1e+16</upper>
+          </limit>
+          <dynamics>
+            <damping>0.00001</damping>
+          </dynamics>
+				</axis>
+	    </joint>
+		</gazebo>
+  </xacro:macro>
 	<xacro:delta_arm
 		parent="base_link"
@@ -198,85 +279,4 @@
 	  <selfCollide>true</selfCollide>
 	</gazebo>
-	<xacro:macro name="link3_with_joint" params="arm_nr suffix sign joint3_type">
-		<joint name="arm${arm_nr}_joint2${suffix}" type="continuous">
-		  <parent link="arm${arm_nr}_link2"/>
-		  <child link="arm${arm_nr}_link3${suffix}"/>
-		  <origin xyz="${sign}0.018 0 0" rpy="0 0 ${-pi/2}"/>
-		  <axis xyz="1 0 0"/>
-		  <dynamics damping="0.00001"/>
-			<xacro:if value="${suffix == '_2'}">
-				<mimic joint="arm${arm_nr}_joint2_1" multiplier="1" offset="0"/>
-			</xacro:if>
-		</joint>
-		<link name="arm${arm_nr}_link3${suffix}">
-		  <visual>
-		    <origin xyz="0 0 0" rpy="0 0 0"/>
-		    <geometry>
-		      <mesh filename="package://eeduro_delta_description/meshes/link3_scaled.dae"/>
-		    </geometry>
-		  </visual>
-			<xacro:link3_inertial/>
-		</link>
-		<xacro:element xacro:name="joint3_${joint3_type}" arm_nr="${arm_nr}" suffix="${suffix}"/>
-	</xacro:macro>
-	<xacro:macro name="joint3_urdf" params="arm_nr suffix">
-			<joint name="arm${arm_nr}_joint3${suffix}" type="continuous">
-			  <parent link="arm${arm_nr}_link3${suffix}"/>
-			  <child link="arm${arm_nr}_link4"/>
-			  <origin xyz="0 0 0.1" rpy="0 0 0"/>
-			  <axis xyz="1 0 0"/>
-			  <dynamics damping="0.00001"/>
-				<mimic joint="arm${arm_nr}_joint2_1" multiplier="-1" offset="0"/>
-			</joint>
-	</xacro:macro>
-	<xacro:macro name="joint3_sdf" params="arm_nr suffix">
-		<gazebo>
-			<joint name="arm${arm_nr}_joint3${suffix}" type="revolute">
-			  <child>arm${arm_nr}_link4</child>
-			  <parent>arm${arm_nr}_link3${suffix}</parent>
-			  <pose>0 -0.036 0 0 0 0</pose>
-			  <axis>
-			    <use_parent_model_frame>false</use_parent_model_frame>
-			    <xyz>1 0 0</xyz>
-			    <limit>
-			      <lower>-1e+16</lower>
-			      <upper>1e+16</upper>
-			    </limit>
-			    <dynamics>
-			      <damping>0.00001</damping>
-			    </dynamics>
-			  </axis>
-			</joint>
-		</gazebo>
-  </xacro:macro>
-	<xacro:macro name="joint4_urdf" params="arm_nr child angle">
-		<joint name="arm${arm_nr}_joint4" type="continuous">
-		  <parent link="arm${arm_nr}_link4"/>
-		  <child link="${child}"/>
-		  <origin xyz="0 -0.018 0" rpy="${angle} 0 ${pi/2}"/>
-		  <axis xyz="1 0 0"/>
-		  <dynamics damping="0.00001"/>
-		</joint>
-	</xacro:macro>
-  <xacro:macro name="joint4_sdf" params="arm_nr child angle">
-    <gazebo>
-			<joint name="arm${arm_nr}_joint4" type="revolute">
-	      <parent>${child}</parent>
-	      <child>arm${arm_nr}_link4</child>
-	      <pose>0 -0.018 0 ${angle} 0 ${pi/2}</pose>
-				<axis>
-          <use_parent_model_frame>false</use_parent_model_frame>
-          <xyz>1 0 0</xyz>
-          <limit>
-            <lower>-1e+16</lower>
-            <upper>1e+16</upper>
-          </limit>
-          <dynamics>
-            <damping>0.00001</damping>
-          </dynamics>
-				</axis>
-	    </joint>
-		</gazebo>
-  </xacro:macro>
 	<gazebo>
 		<plugin name="gazebo_ros_joint_state_publisher" filename="libgazebo_ros_joint_state_publisher.so">
